File: MyMouse/MyMouse.kicad_pcb (KiCad board)
At the start: 2 copper layers, 13 parts, among them J1 Conn_01x04, SW1 SW_Push, SW10 SW_Push, SW2 SW_Push, SW3 SW_Push, SW4 SW_Push, SW5 SW_Push, SW6 SW_Push, SW8 RotaryEncoder_Switch, SW9 RotaryEncoder_Switch

Commit message: 進めた
Parts:
- added U1: PMW3360DM-T2QU, PMW3360_PCB:PMW3360DM-T2QU 16Pin, F.Cu at (96.8, 78.8)
- moved D1 148.3 mm to (81.6, 79.8), turned to 90 degrees
- moved SW9 129.1 mm to (96.8, 48.2), turned to -90 degrees
- moved BT1 127.0 mm to (97.8, 92.2), turned to 90 degrees
- moved SW1 126.0 mm to (67.5, 23.0)
- moved J1 118.4 mm to (120.2, 75.2)
- moved SW10 101.8 mm to (109.8, 53.8)
- moved SW2 99.3 mm to (117.0, 23.0)
- moved A1 96.7 mm to (201.3, 58.6)
- moved SW6 96.6 mm to (263.9, 39.8), turned to -90 degrees
- moved SW5 90.4 mm to (264.9, 31.2), turned to 180 degrees
- moved SW3 41.8 mm to (135.8, 32.2)
- moved SW8 40.3 mm to (259.9, 69.0), turned to 90 degrees
- moved SW4 38.5 mm to (145.2, 50.2)
Other:
- board outline added: 212.5 x 103.5 mm
